Commit message: Start setting up visualization

File: catkin_ws/src/aquadrone_description/urdf/aquadrone_v2.urdf.xacro (robot description, xacro)
@@ -112,4 +112,14 @@
         </link>
       </plugin>
+    <plugin name="p3d_base_controller" filename="libgazebo_ros_p3d.so">
+      <alwaysOn>true</alwaysOn>
+      <updateRate>50.0</updateRate>
+      <bodyName>base_link</bodyName>
+      <topicName>/aquadrone/internal/sim_only/global_pos</topicName>
+      <gaussianNoise>0.01</gaussianNoise>
+      <frameName>world</frameName>
+      <xyzOffsets>0 0 0</xyzOffsets>
+      <rpyOffsets>0 0 0</rpyOffsets>
+    </plugin>
     </gazebo>
   </xacro:macro>

File: catkin_ws/src/aquadrone_description/urdf/thruster.urdf.xacro (robot description, xacro)
@@ -30,4 +30,14 @@
       <child link="thruster_${thruster_id}" />
     </joint>
+    <transmission name="thruster_${thruster_id}_transmission" type="SimpleTransmission">
+      <type>transmission_interface/SimpleTransmission</type>
+      <joint name="thruster_${thruster_id}_joint">
+        <hardwareInterface>EffortJointInterface</hardwareInterface>
+      </joint>
+      <actuator name="thruster_${thruster_id}_joint_motor">
+        <hardwareInterface>EffortJointInterface</hardwareInterface>
+        <mechanicalReduction>1</mechanicalReduction>
+      </actuator>
+    </transmission>
     <gazebo>
       <!-- Thruster ROS plugin -->
